File: kicad/v1.2/Logic.kicad_sch (KiCad schematic)
At the start: 30 parts, among them J1 JTAG, J1 MZ-700 Bus, J2 FDC-34, J4 Floppy Power Connector, Q1 C945, U1 74LS06, U13 WD1773, U2 74LS04, U4 74LS14, U4 EPM7128SLC84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

Commit message: Added GAL compiled files
Parts:
- renumbered C15 to C10, C4 to C11, C17 to C12, C8 to C13, C8 to C14, C8 to C15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
