File: kicad/v1.2/PowerDecoupling.kicad_sch (KiCad schematic)
At the start: 13 parts, among them U1 74LS06, U15 EPM7128SLC84, U2 74LS04, U4 74LS14

Commit message: Added GAL compiled files
Parts:
- renumbered C5 to C3, C6 to C4, C7 to C5, C7 to C6, C7 to C8, C7 to C9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
